File: CompletePCB.sch (EAGLE design)
At the start: 86 parts, among them IC1 SA602AD_01,118, IC3 L78L08ABUTR, IC4 LM386M-1, T1 2N3565, T2 2N3565, T3 2N3565, T4 2N3565, T5 2N3565, X1 1-227161-0

Commit message: Changes Made over time
Parts:
- removed C37: GKG20015, SamacSys_Parts:GKG20015
- removed X1: 1-227161-0, con-coax:1-227161-0
- added C19, C25: (no value), eagle-ltspice:C
- added J1: 5413631-1, SamacSys_Parts:5413631-1
- added R22, R23, R24, R25: (no value), resistor:R-US_R0805
- added T6: 2N3565, transistor:2N3565
- C26: value GKG20015 -> (none); device SamacSys_Parts:GKG20015 -> eagle-ltspice:C
- U$10: value WOUNDINDUCTOR -> 42IF123; device Custom:WOUNDINDUCTOR -> Custom:42IF123
- U$3: value RFTRANSFORMER -> 42IF123; device Custom:RFTRANSFORMER -> Custom:42IF123
Connections:
- new net N$2: C30.+, C31.2, IC3.VOUT, U$18.2
- new net N$34: C19.1, IC1.VCC, U$18.1
- new net N$37: R24.2, T6.E
- new net N$38: C25.1, R24.1, R25.2
- new net N$43: C13.2, U$14.1, U$15.2
- net GND: now also C19.2, C25.2, J1.2, J1.3, J1.4, J1.5, R23.1, R25.1, U$10.P$5, U$3.P$3; no longer C13.2, C26.1, U$10.1, U$18.1, U$3.P$1, X1.2
- net IF: now also U$3.P$4; no longer U$3.P$2
- net N$15: now also J1.1; no longer U$14.1, U$15.2, X1.1
- net N$20: now also U$3.P$1; no longer C37.2, U$3.P$3
- net N$21: now also U$3.P$5; no longer C37.1, U$3.P$4
- net N$26: now also T6.C; no longer T3.C
- net N$27: now also U$10.P$1; no longer C26.2, U$10.2
- net N$39: now also C26.1, R13.2, T3.E; no longer C30.+, C31.2, IC1.VCC, IC3.VOUT, U$18.2
- net N$6: now also C26.2, R22.1, R23.2, T6.B; no longer R13.2, T3.E
- net VCC: now also R22.2, T3.C
Other:
- moved on the sheet: C13, C20, C21, C22, C28, R11, R12, R13, R14, T3, U$11, U$12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
